Commit message: tidied up gazebo launch code

File: tracebot_mockup_gazebo/urdf/tracebot_mockup.urdf.xacro (robot description, xacro)
@@ -1,41 +1,20 @@
 <?xml version="1.0"?>
-<robot xmlns:xacro="http://wiki.ros.org/xacro" name="ur_robot_gazebo">
-  <!--
-    This is a top-level xacro instantiating the Gazebo-specific version of the
-    'ur_robot' macro (ie: 'ur_robot_gazebo') and passing it values for all its
-    required arguments.
-    This file should be considered the Gazebo-specific variant of the file
-    with the same name in the ur_description package. It accepts the same
-    arguments, but instead of configuring everything for a real robot, will
-    generate a Gazebo-compatible URDF with a ros_control hardware_interface
-    attached to it.
-    Only use this top-level xacro if you plan on spawning the robot in Gazebo
-    'by itself', without any gripper or any other geometry attached.
-    If you need to attach an end-effector, camera or need to integrate the
-    robot into a larger workcell and want to spawn that as a single entity in
-    Gazebo, DO NOT EDIT THIS FILE.
-    Instead: create a new top-level xacro, give it a proper name, include the
-    required '.xacro' files, instantiate the models (ie: call the macros) and
-    connect everything by adding the appropriate joints.
-  -->
-  <!--
-    Import main macro.
-    NOTE: this imports the Gazebo-wrapper main macro, NOT the regular
-          xacro macro (which is hosted by ur_description).
-  -->
-  <xacro:include filename="$(find tracebot_mockup_gazebo)/urdf/ur_macro.xacro"/>
+<robot xmlns:xacro="http://wiki.ros.org/xacro" name="tracebot_mockup_gazebo">
   <xacro:include filename="$(find tracebot_mockup_gazebo)/urdf/tracebot_mockup_macro.urdf.xacro"/>
-  <!--
-    legal values:
-      - hardware_interface/PositionJointInterface
-      - hardware_interface/VelocityJointInterface
-      - hardware_interface/EffortJointInterface
-    NOTE: this value must correspond to the controller configured in the
-          controller .yaml files in the 'config' directory.
-  -->
+  <xacro:include filename="$(find ur_gazebo)/urdf/ur_macro.xacro"/>
+  <!--Robot base parameters-->
+  <xacro:arg name="robot_mount_offset_x" default="0.1293"/>
+  <xacro:arg name="robot_mount_offset_y" default="0.0"/>
+  <xacro:arg name="robot_mount_offset_z" default="0.0707"/>
+  <xacro:arg name="robot_mount_offset_theta" default="0.0"/>
+  <xacro:arg name="robot_mount_length" default="0.55"/>
+  <xacro:arg name="robot_mount_width" default="0.55"/>
+  <xacro:arg name="robot_mount_height" default="1.2664"/>
+  <xacro:arg name="robot_base_tilt" default="0.785398"/>
+  <xacro:arg name="left_arm" default="ur5e"/>
+  <xacro:arg name="right_arm" default="ur5e"/>
+  <!--Robot arm parameters-->
   <xacro:arg name="transmission_hw_interface" default="hardware_interface/PositionJointInterface"/>
-  <xacro:arg name="safety_limits" default="false"/>
-  <xacro:arg name="safety_pos_margin" default="0.15"/>
-  <xacro:arg name="safety_k_position" default="20"/>
+  <!--Add parameters to robot base-->
   <xacro:tracebot_mockup_gazebo
     robot_mount_offset_x="$(arg robot_mount_offset_x)"
@@ -49,7 +28,16 @@
     left_arm="$(arg left_arm)"
     right_arm="$(arg right_arm)"/>
-  <!-- Instantiate the Gazebo robot and pass it all the required arguments. -->
-  <xacro:ur_robot_gazebo
-    prefix="right_"
+  <!--Add parameters to robot arms-->
+  <xacro:ur_robot_gazebo prefix="left_"
+    joint_limits_parameters_file="$(find ur_description)/config/$(arg left_arm)/joint_limits.yaml"
+    kinematics_parameters_file="$(find ur_description)/config/$(arg left_arm)/default_kinematics.yaml"
+    physical_parameters_file="$(find ur_description)/config/$(arg left_arm)/physical_parameters.yaml"
+    visual_parameters_file="$(find ur_description)/config/$(arg left_arm)/visual_parameters.yaml"
+    transmission_hw_interface="$(arg transmission_hw_interface)"
+    safety_limits="false"
+    safety_pos_margin="0.15"
+    safety_k_position="20"/>
+    <xacro:ur_arm_transmission prefix="left_" hw_interface="$(arg transmission_hw_interface)" />
+  <xacro:ur_robot_gazebo prefix="right_"
     joint_limits_parameters_file="$(find ur_description)/config/$(arg right_arm)/joint_limits.yaml"
     kinematics_parameters_file="$(find ur_description)/config/$(arg right_arm)/default_kinematics.yaml"
@@ -59,24 +47,12 @@
     safety_limits="false"
     safety_pos_margin="0.15"
-    safety_k_position="20"
-  />
-  <xacro:ur_robot_gazebo
-    prefix="left_"
-    joint_limits_parameters_file="$(find ur_description)/config/$(arg right_arm)/joint_limits.yaml"
-    kinematics_parameters_file="$(find ur_description)/config/$(arg right_arm)/default_kinematics.yaml"
-    physical_parameters_file="$(find ur_description)/config/$(arg right_arm)/physical_parameters.yaml"
-    visual_parameters_file="$(find ur_description)/config/$(arg right_arm)/visual_parameters.yaml"
-    transmission_hw_interface="$(arg transmission_hw_interface)"
-    safety_limits="false"
-    safety_pos_margin="0.15"
-    safety_k_position="20"
-  />
-  <!--
-    Attach the Gazebo model to Gazebo's world frame.
-    Note: if you're looking to integrate a UR into a larger scene and need
-    to add EEFs or other parts, DO NOT change this file or the 'world' link
-    here. Create a NEW xacro instead and decide whether you need to add
-    a 'world' link there.
-  -->
+    safety_k_position="20"/>
+  <xacro:ur_arm_transmission prefix="right_" hw_interface="$(arg transmission_hw_interface)" />
+  <!--Link arms to base-->
+  <joint name="left_base_link_joint" type="fixed">
+    <origin xyz="0 0 0" rpy="0 0 0"/>
+    <parent link="left_robot_mount"/>
+    <child link="left_base_link"/>
+  </joint>
   <joint name="right_base_link_joint" type="fixed">
     <origin xyz="0 0 0" rpy="0 0 0"/>
@@ -84,9 +60,5 @@
     <child link="right_base_link"/>
   </joint>
-  <joint name="left_base_link_joint" type="fixed">
-    <origin xyz="0 0 0" rpy="0 0 0"/>
-    <parent link="left_robot_mount"/>
-    <child link="left_base_link"/>
-  </joint>
+  <!--Link base to world-->
   <link name="world"/>
   <joint name="world_joint" type="fixed">
@@ -95,9 +67,3 @@
     <origin xyz="0 0 0" rpy="0 0 0"/>
   </joint>
-    <gazebo>
-      <plugin name="ros_control" filename="libgazebo_ros_control.so">
-        <!--robotNamespace>/</robotNamespace-->
-        <!--robotSimType>gazebo_ros_control/DefaultRobotHWSim</robotSimType-->
-      </plugin>
-    </gazebo>
 </robot>

File: tracebot_mockup_gazebo/urdf/tracebot_mockup_macro.urdf.xacro (robot description, xacro)
@@ -13,4 +13,5 @@
     right_arm">
     <xacro:include filename="$(find tracebot_mockup_description)/urdf/tracebot_mockup_macro.urdf.xacro"/>
+    <!--Pass arguments to tracebot_mockup-->
     <xacro:tracebot_mockup
       robot_mount_offset_x="${robot_mount_offset_x}"
@@ -25,4 +26,5 @@
       right_arm="${right_arm}"
     />
+    <!--Add collision to base-->
     <gazebo reference="robot_mount_base">
       <selfCollide>true</selfCollide>

Commit message: Added single arm functionality in gazebo

File: tracebot_mockup_gazebo/urdf/tracebot_mockup.urdf.xacro (robot description, xacro)
@@ -38,5 +38,5 @@
     safety_pos_margin="0.15"
     safety_k_position="20"/>
-  <xacro:ur_robot_gazebo prefix="right_"
+  <!--xacro:ur_robot_gazebo prefix="right_"
     joint_limits_parameters_file="$(find ur_description)/config/$(arg right_arm)/joint_limits.yaml"
     kinematics_parameters_file="$(find ur_description)/config/$(arg right_arm)/default_kinematics.yaml"
@@ -46,5 +46,5 @@
     safety_limits="false"
     safety_pos_margin="0.15"
-    safety_k_position="20"/>
+    safety_k_position="20"/-->
   <!--Link arms to base-->
   <joint name="left_base_link_joint" type="fixed">
@@ -53,9 +53,9 @@
     <child link="left_base_link"/>
   </joint>
-  <joint name="right_base_link_joint" type="fixed">
+  <!--joint name="right_base_link_joint" type="fixed">
     <origin xyz="0 0 0" rpy="0 0 -1.5708"/>
     <parent link="right_robot_mount"/>
     <child link="right_base_link"/>
-  </joint>
+  </joint-->
   <!--Link base to world-->
   <link name="world"/>

Commit message: Added functionality for both arms

File: tracebot_mockup_gazebo/urdf/tracebot_mockup.urdf.xacro (robot description, xacro)
@@ -2,5 +2,5 @@
 <robot xmlns:xacro="http://wiki.ros.org/xacro" name="tracebot_mockup_gazebo">
   <xacro:include filename="$(find tracebot_mockup_gazebo)/urdf/tracebot_mockup_macro.urdf.xacro"/>
-  <xacro:include filename="$(find ur_gazebo)/urdf/ur_macro.xacro"/>
+  <xacro:include filename="$(find tracebot_mockup_gazebo)/urdf/ur_macro.xacro"/>
   <!--Robot base parameters-->
   <xacro:arg name="robot_mount_offset_x" default="0.1293"/>
@@ -38,5 +38,5 @@
     safety_pos_margin="0.15"
     safety_k_position="20"/>
-  <!--xacro:ur_robot_gazebo prefix="right_"
+  <xacro:ur_robot_gazebo prefix="right_"
     joint_limits_parameters_file="$(find ur_description)/config/$(arg right_arm)/joint_limits.yaml"
     kinematics_parameters_file="$(find ur_description)/config/$(arg right_arm)/default_kinematics.yaml"
@@ -46,5 +46,5 @@
     safety_limits="false"
     safety_pos_margin="0.15"
-    safety_k_position="20"/-->
+    safety_k_position="20"/>
   <!--Link arms to base-->
   <joint name="left_base_link_joint" type="fixed">
@@ -53,9 +53,9 @@
     <child link="left_base_link"/>
   </joint>
-  <!--joint name="right_base_link_joint" type="fixed">
+  <joint name="right_base_link_joint" type="fixed">
     <origin xyz="0 0 0" rpy="0 0 -1.5708"/>
     <parent link="right_robot_mount"/>
     <child link="right_base_link"/>
-  </joint-->
+  </joint>
   <!--Link base to world-->
   <link name="world"/>
@@ -65,3 +65,9 @@
     <origin xyz="0 0 0" rpy="0 0 0"/>
   </joint>
+  <gazebo>
+    <plugin name="ros_control" filename="libgazebo_ros_control.so">
+      <!--robotNamespace>/</robotNamespace-->
+      <!--robotSimType>gazebo_ros_control/DefaultRobotHWSim</robotSimType-->
+    </plugin>
+  </gazebo>
 </robot>
