Commit message: Add parameters to change robot_mount and pump position on table

File: tracebot_mockup_description/urdf/tracebot_mockup.urdf.xacro (robot description, xacro)
@@ -4,7 +4,13 @@
   <xacro:arg name="table_width" default="2.0"/>
   <xacro:arg name="table_height" default="1.0"/>
+  <xacro:arg name="robot_mount_offset_x" default="0.0"/>
+  <xacro:arg name="robot_mount_offset_y" default="-0.2"/>
+  <xacro:arg name="robot_mount_offset_theta" default="0.0"/>
   <xacro:arg name="robot_mount_length" default="0.2"/>
   <xacro:arg name="robot_mount_width" default="0.2"/>
   <xacro:arg name="robot_mount_height" default="0.6"/>
+  <xacro:arg name="pump_offset_x" default="0.0"/>
+  <xacro:arg name="pump_offset_y" default="0.2"/>
+  <xacro:arg name="pump_offset_theta" default="0.0"/>
   <xacro:arg name="pump_length" default="0.2"/>
   <xacro:arg name="pump_width" default="0.3"/>
@@ -14,7 +20,13 @@
     table_width="$(arg table_width)"
     table_height="$(arg table_height)"
+    robot_mount_offset_x="$(arg robot_mount_offset_x)"
+    robot_mount_offset_y="$(arg robot_mount_offset_y)"
+    robot_mount_offset_theta="$(arg robot_mount_offset_theta)"
     robot_mount_length="$(arg robot_mount_length)"
     robot_mount_width="$(arg robot_mount_width)"
     robot_mount_height="$(arg robot_mount_height)"
+    pump_offset_x="$(arg pump_offset_x)"
+    pump_offset_y="$(arg pump_offset_y)"
+    pump_offset_theta="$(arg pump_offset_theta)"
     pump_length="$(arg pump_length)"
     pump_width="$(arg pump_width)"

File: tracebot_mockup_description/urdf/tracebot_mockup_macro.urdf.xacro (robot description, xacro)
@@ -5,7 +5,13 @@
                                               table_length
                                               table_width
+                                              robot_mount_offset_x
+                                              robot_mount_offset_y
+                                              robot_mount_offset_theta
                                               robot_mount_height
                                               robot_mount_length
                                               robot_mount_width
+                                              pump_offset_x
+                                              pump_offset_y
+                                              pump_offset_theta
                                               pump_height
                                               pump_length
@@ -40,5 +46,5 @@
     </link>
     <joint name="robot_mount_base_joint" type="fixed">
-      <origin xyz="0 0 0" rpy="0 0 0"/>
+      <origin xyz="${robot_mount_offset_x} ${robot_mount_offset_y} 0" rpy="0 0 ${robot_mount_offset_theta}"/>
       <parent link="table"/>
       <child link="robot_mount_base"/>
@@ -96,5 +102,5 @@
     </link>
     <joint name="pump_joint" type="fixed">
-      <origin xyz="0 0.5 0" rpy="0 0 0"/>
+      <origin xyz="${pump_offset_x} ${pump_offset_y} 0" rpy="0 0 ${pump_offset_theta}"/>
       <parent link="table"/>
       <child link="pump"/>

Commit message: Add parameter to tilt robot base

File: tracebot_mockup_description/urdf/tracebot_mockup.urdf.xacro (robot description, xacro)
@@ -11,4 +11,5 @@
     robot_mount_width="$(arg robot_mount_width)"
     robot_mount_height="$(arg robot_mount_height)"
+    robot_base_tilt="$(arg robot_base_tilt)"
     pump_offset_x="$(arg pump_offset_x)"
     pump_offset_y="$(arg pump_offset_y)"

File: tracebot_mockup_description/urdf/tracebot_mockup_macro.urdf.xacro (robot description, xacro)
@@ -11,4 +11,5 @@
                                               robot_mount_length
                                               robot_mount_width
+                                              robot_base_tilt
                                               pump_offset_x
                                               pump_offset_y
@@ -52,5 +53,5 @@
     <link name="left_robot_mount"/>
     <joint name="left_robot_mount_joint" type="fixed">
-      <origin xyz="${robot_mount_length/2} 0 ${robot_mount_height/2}" rpy="0 ${pi/2} 0"/>
+      <origin xyz="${robot_mount_length/2} 0 ${robot_mount_height/2}" rpy="0 ${pi/2 - robot_base_tilt} 0"/>
       <parent link="robot_mount_base"/>
       <child link="left_robot_mount"/>
@@ -58,5 +59,5 @@
     <link name="right_robot_mount"/>
     <joint name="right_robot_mount_joint" type="fixed">
-      <origin xyz="${-robot_mount_length/2} 0 ${robot_mount_height/2}" rpy="0 ${-pi/2} 0"/>
+      <origin xyz="${-robot_mount_length/2} 0 ${robot_mount_height/2}" rpy="0 ${-pi/2 + robot_base_tilt} 0"/>
       <parent link="robot_mount_base"/>
       <child link="right_robot_mount"/>

Commit message: Added motor control to gazebo

File: tracebot_mockup_description/urdf/tracebot_mockup.urdf.xacro (robot description, xacro)
@@ -2,9 +2,9 @@
 <robot xmlns:xacro="http://wiki.ros.org/xacro" name="ur">
   <xacro:include filename="$(find tracebot_mockup_description)/urdf/tracebot_mockup_macro.urdf.xacro"/>
-  <xacro:tracebot_mockup table_length="$(arg table_length)"
-    table_width="$(arg table_width)"
-    table_height="$(arg table_height)"
+  <xacro:include filename="$(find ur_description)/urdf/ur_macro.xacro"/>
+  <xacro:tracebot_mockup
     robot_mount_offset_x="$(arg robot_mount_offset_x)"
     robot_mount_offset_y="$(arg robot_mount_offset_y)"
+    robot_mount_offset_z="$(arg robot_mount_offset_z)"
     robot_mount_offset_theta="$(arg robot_mount_offset_theta)"
     robot_mount_length="$(arg robot_mount_length)"
@@ -12,11 +12,34 @@
     robot_mount_height="$(arg robot_mount_height)"
     robot_base_tilt="$(arg robot_base_tilt)"
-    pump_offset_x="$(arg pump_offset_x)"
-    pump_offset_y="$(arg pump_offset_y)"
-    pump_offset_theta="$(arg pump_offset_theta)"
-    pump_length="$(arg pump_length)"
-    pump_width="$(arg pump_width)"
-    pump_height="$(arg pump_height)"
     left_arm="$(arg left_arm)"
     right_arm="$(arg right_arm)"/>
+  <xacro:ur_robot prefix=""
+    joint_limits_parameters_file="$(find ur_description)/config/$(arg left_arm)/joint_limits.yaml"
+    kinematics_parameters_file="$(find ur_description)/config/$(arg left_arm)/default_kinematics.yaml"
+    physical_parameters_file="$(find ur_description)/config/$(arg left_arm)/physical_parameters.yaml"
+    visual_parameters_file="$(find ur_description)/config/$(arg left_arm)/visual_parameters.yaml"
+    transmission_hw_interface="hardware_interface/VelocityJointInterface"
+    safety_limits="false"
+    safety_pos_margin="0.15"
+    safety_k_position="20"/>
+  <xacro:ur_robot prefix="right_"
+    joint_limits_parameters_file="$(find ur_description)/config/$(arg right_arm)/joint_limits.yaml"
+    kinematics_parameters_file="$(find ur_description)/config/$(arg right_arm)/default_kinematics.yaml"
+    physical_parameters_file="$(find ur_description)/config/$(arg right_arm)/physical_parameters.yaml"
+    visual_parameters_file="$(find ur_description)/config/$(arg right_arm)/visual_parameters.yaml"
+    transmission_hw_interface="hardware_interface/VelocityJointInterface"
+    safety_limits="false"
+    safety_pos_margin="0.15"
+    safety_k_position="20"/>
+  <!-- Attach arms to base -->
+  <joint name="base_link_joint" type="fixed">
+    <origin xyz="0 0 0" rpy="0 0 0"/>
+    <parent link="left_robot_mount"/>
+    <child link="base_link"/>
+  </joint>
+  <joint name="right_base_link_joint" type="fixed">
+    <origin xyz="0 0 0" rpy="0 0 0"/>
+    <parent link="right_robot_mount"/>
+    <child link="right_base_link"/>
+  </joint>
 </robot>

File: tracebot_mockup_description/urdf/tracebot_mockup_macro.urdf.xacro (robot description, xacro)
@@ -1,11 +1,9 @@
 <?xml version="1.0"?>
 <robot xmlns:xacro="http://wiki.ros.org/xacro">
-  <xacro:include filename="$(find ur_description)/urdf/ur_macro.xacro"/>
   <xacro:macro name="tracebot_mockup"
-    params="table_height
-    table_length
-    table_width
+    params="
     robot_mount_offset_x
     robot_mount_offset_y
+    robot_mount_offset_z
     robot_mount_offset_theta
     robot_mount_height
@@ -13,32 +11,15 @@
     robot_mount_width
     robot_base_tilt
-    pump_offset_x
-    pump_offset_y
-    pump_offset_theta
-    pump_height
-    pump_length
-    pump_width
     left_arm
     right_arm">
-    <link name="base_link"/>
-    <link name="table">
-      <visual>
-        <origin xyz="0 0 0.525" rpy="0 0 0"/>
-        <geometry>
-          <mesh filename="file:///home/benrjg/astech_wss/tracebot_mockup_ws/src/tracebot_mockup/tracebot_mockup_description/meshes/table.stl" />
-        </geometry>
-        <material name="grey">
-          <color rgba="0.6 0.6 0.6 1.0"/>
-        </material>
-      </visual>
-    </link>
-    <joint name="table_joint" type="fixed">
+    <link name="robot_base_link"/>
+    <joint name="robot_mount_base_joint" type="fixed">
       <origin xyz="0 0 0" rpy="0 0 0"/>
-      <parent link="base_link"/>
-      <child link="table"/>
+      <parent link="robot_base_link"/>
+      <child link="robot_mount_base"/>
     </joint>
     <link name="robot_mount_base">
       <visual>
-        <origin xyz="0 0 0.6332" rpy="0 0 0"/>
+        <origin xyz="0 0 ${robot_mount_height/2}" rpy="0 0 0"/>
         <geometry>
           <mesh filename="file:///home/benrjg/astech_wss/tracebot_mockup_ws/src/tracebot_mockup/tracebot_mockup_description/meshes/stand.stl" />
@@ -49,65 +30,18 @@
       </visual>
     </link>
-    <joint name="robot_mount_base_joint" type="fixed">
-      <origin xyz="0 -0.45 0" rpy="0 0 0"/>
-      <parent link="base_link"/>
-      <child link="robot_mount_base"/>
-    </joint>
-    <link name="left_robot_mount"/>
+    <!-- Left Arm Mount -->
     <joint name="left_robot_mount_joint" type="fixed">
-      <origin xyz="-0.1293 0 1.1957" rpy="0 ${-1.57079632679+robot_base_tilt} 0"/>
+      <origin xyz="${-robot_mount_offset_x} 0 ${robot_mount_height-robot_mount_offset_z}" rpy="0 ${-pi/2+robot_base_tilt} 0"/>
       <parent link="robot_mount_base"/>
       <child link="left_robot_mount"/>
     </joint>
-    <link name="right_robot_mount"/>
+    <link name="left_robot_mount"/>
+    <!-- Right Arm Mount -->
     <joint name="right_robot_mount_joint" type="fixed">
-      <origin xyz="0.1293 0 1.1957" rpy="0 ${1.57079632679-robot_base_tilt} 0"/>
+      <origin xyz="${robot_mount_offset_x} 0 ${robot_mount_height-robot_mount_offset_z}" rpy="0 ${pi/2-robot_base_tilt} 0"/>
       <parent link="robot_mount_base"/>
       <child link="right_robot_mount"/>
     </joint>
-    <xacro:ur_robot prefix="left_"
-      joint_limits_parameters_file="$(find ur_description)/config/${left_arm}/joint_limits.yaml"
-                    kinematics_parameters_file="$(find ur_description)/config/${left_arm}/default_kinematics.yaml"
-                    physical_parameters_file="$(find ur_description)/config/${left_arm}/physical_parameters.yaml"
-                    visual_parameters_file="$(find ur_description)/config/${left_arm}/visual_parameters.yaml"
-                    transmission_hw_interface="hardware_interface/VelocityJointInterface"
-                    safety_limits="false"
-                    safety_pos_margin="0.15"
-                    safety_k_position="20"/>
-    <joint name="left_base_link_joint" type="fixed">
-      <origin xyz="0 0 0" rpy="0 0 0"/>
-      <parent link="left_robot_mount"/>
-      <child link="left_base_link"/>
-    </joint>
-    <xacro:ur_robot prefix="right_"
-      joint_limits_parameters_file="$(find ur_description)/config/${right_arm}/joint_limits.yaml"
-                    kinematics_parameters_file="$(find ur_description)/config/${right_arm}/default_kinematics.yaml"
-                    physical_parameters_file="$(find ur_description)/config/${right_arm}/physical_parameters.yaml"
-                    visual_parameters_file="$(find ur_description)/config/${right_arm}/visual_parameters.yaml"
-                    transmission_hw_interface="hardware_interface/VelocityJointInterface"
-                    safety_limits="false"
-                    safety_pos_margin="0.15"
-                    safety_k_position="20"/>
-    <joint name="right_base_link_joint" type="fixed">
-      <origin xyz="0 0 0" rpy="0 0 0"/>
-      <parent link="right_robot_mount"/>
-      <child link="right_base_link"/>
-    </joint>
-    <link name="pump">
-      <visual>
-        <origin xyz="0 0 0" rpy="0 0 0"/>
-        <geometry>
-          <mesh filename="file:///home/benrjg/astech_wss/tracebot_mockup_ws/src/tracebot_mockup/tracebot_mockup_description/meshes/pump.stl" />
-        </geometry>
-        <material name="pink">
-          <color rgba="1.0 0.0 1.0 1.0"/>
-        </material>
-      </visual>
-    </link>
-    <joint name="pump_joint" type="fixed">
-      <origin xyz="0 0.2 1.05" rpy="1.5708 0 0"/>
-      <parent link="table"/>
-      <child link="pump"/>
-    </joint>
+    <link name="right_robot_mount"/>
   </xacro:macro>
 </robot>

File: tracebot_mockup_gazebo/urdf/tracebot_mockup.urdf.xacro (robot description, xacro)
@@ -3,28 +3,23 @@
   <xacro:include filename="$(find tracebot_mockup_gazebo)/urdf/tracebot_mockup_macro.urdf.xacro"/>
   <xacro:include filename="$(find tracebot_mockup_description)/urdf/tracebot_mockup_macro.urdf.xacro"/>
+  <xacro:include filename="$(find ur_gazebo)/urdf/ur_macro.xacro"/>
+  <xacro:include filename="$(find ur_description)/urdf/inc/ur_transmissions.xacro" />
+  <xacro:include filename="$(find ur_description)/urdf/inc/ur_common.xacro" />
   <xacro:arg name="joint_limit_params" default=""/>
-  <xacro:arg name="table_length" default="2.0"/>
-  <xacro:arg name="table_width" default="2.0"/>
-  <xacro:arg name="table_height" default="1.0"/>
-  <xacro:arg name="robot_mount_offset_x" default="0.0"/>
-  <xacro:arg name="robot_mount_offset_y" default="-0.2"/>
+  <xacro:arg name="robot_mount_offset_x" default="0.1293"/>
+  <xacro:arg name="robot_mount_offset_y" default="0.0"/>
+  <xacro:arg name="robot_mount_offset_z" default="0.0707"/>
   <xacro:arg name="robot_mount_offset_theta" default="0.0"/>
-  <xacro:arg name="robot_mount_length" default="0.2"/>
-  <xacro:arg name="robot_mount_width" default="0.2"/>
-  <xacro:arg name="robot_mount_height" default="0.6"/>
-  <xacro:arg name="robot_base_tilt" default="0.0"/>
-  <xacro:arg name="pump_offset_x" default="0.0"/>
-  <xacro:arg name="pump_offset_y" default="0.2"/>
-  <xacro:arg name="pump_offset_theta" default="0.0"/>
-  <xacro:arg name="pump_length" default="0.2"/>
-  <xacro:arg name="pump_width" default="0.0"/>
-  <xacro:arg name="pump_height" default="0.0"/>
+  <xacro:arg name="robot_mount_length" default="0.55"/>
+  <xacro:arg name="robot_mount_width" default="0.55"/>
+  <xacro:arg name="robot_mount_height" default="1.2664"/>
+  <xacro:arg name="robot_base_tilt" default="0.785398"/>
   <xacro:arg name="left_arm" default="ur5e"/>
   <xacro:arg name="right_arm" default="ur5e"/>
-  <xacro:tracebot_mockup_gazebo table_length="$(arg table_length)"
-    table_width="$(arg table_width)"
-    table_height="$(arg table_height)"
+  <xacro:arg name="transmission_hw_interface" default="hardware_interface/PositionJointInterface"/>
+  <xacro:tracebot_mockup_gazebo
     robot_mount_offset_x="$(arg robot_mount_offset_x)"
     robot_mount_offset_y="$(arg robot_mount_offset_y)"
+    robot_mount_offset_z="$(arg robot_mount_offset_z)"
     robot_mount_offset_theta="$(arg robot_mount_offset_theta)"
     robot_mount_length="$(arg robot_mount_length)"
@@ -32,16 +27,43 @@
     robot_mount_height="$(arg robot_mount_height)"
     robot_base_tilt="$(arg robot_base_tilt)"
-    pump_offset_x="$(arg pump_offset_x)"
-    pump_offset_y="$(arg pump_offset_y)"
-    pump_offset_theta="$(arg pump_offset_theta)"
-    pump_length="$(arg pump_length)"
-    pump_width="$(arg pump_width)"
-    pump_height="$(arg pump_height)"
     left_arm="$(arg left_arm)"
     right_arm="$(arg right_arm)"/>
+  <xacro:ur_robot_gazebo prefix=""
+    joint_limits_parameters_file="$(find ur_description)/config/$(arg left_arm)/joint_limits.yaml"
+    kinematics_parameters_file="$(find ur_description)/config/$(arg left_arm)/default_kinematics.yaml"
+    physical_parameters_file="$(find ur_description)/config/$(arg left_arm)/physical_parameters.yaml"
+    visual_parameters_file="$(find ur_description)/config/$(arg left_arm)/visual_parameters.yaml"
+    transmission_hw_interface="hardware_interface/VelocityJointInterface"
+    safety_limits="false"
+    safety_pos_margin="0.15"
+    safety_k_position="20"/>
+    <!-- Add URDF transmission elements (for ros_control) -->
+    <xacro:ur_arm_transmission prefix="" hw_interface="$(arg transmission_hw_interface)" />
+  <xacro:ur_robot_gazebo prefix="right_"
+    joint_limits_parameters_file="$(find ur_description)/config/$(arg right_arm)/joint_limits.yaml"
+    kinematics_parameters_file="$(find ur_description)/config/$(arg right_arm)/default_kinematics.yaml"
+    physical_parameters_file="$(find ur_description)/config/$(arg right_arm)/physical_parameters.yaml"
+    visual_parameters_file="$(find ur_description)/config/$(arg right_arm)/visual_parameters.yaml"
+    transmission_hw_interface="hardware_interface/VelocityJointInterface"
+    safety_limits="false"
+    safety_pos_margin="0.15"
+    safety_k_position="20"/>
+  <!-- Add URDF transmission elements (for ros_control) -->
+  <xacro:ur_arm_transmission prefix="right_" hw_interface="$(arg transmission_hw_interface)" />
+  <!-- Attach arms to base -->
+  <joint name="left_base_link_joint" type="fixed">
+    <origin xyz="0 0 0" rpy="0 0 0"/>
+    <parent link="left_robot_mount"/>
+    <child link="base_link"/>
+  </joint>
+  <joint name="right_base_link_joint" type="fixed">
+    <origin xyz="0 0 0" rpy="0 0 0"/>
+    <parent link="right_robot_mount"/>
+    <child link="right_base_link"/>
+  </joint>
   <link name="world"/>
   <joint name="world_joint" type="fixed">
     <parent link="world"/>
-    <child link="base_link"/>
+    <child link="robot_base_link"/>
     <origin xyz="0 0 0" rpy="0 0 0"/>
   </joint>

File: tracebot_mockup_gazebo/urdf/tracebot_mockup_macro.urdf.xacro (robot description, xacro)
@@ -1,11 +1,10 @@
 <?xml version="1.0"?>
 <robot xmlns:xacro="http://wiki.ros.org/xacro">
-  <xacro:include filename="$(find ur_description)/urdf/ur_macro.xacro"/>
+  <xacro:include filename="$(find tracebot_mockup_description)/urdf/tracebot_mockup_macro.urdf.xacro"/>
   <xacro:macro name="tracebot_mockup_gazebo"
-    params="table_height
-    table_length
-    table_width
+    params="
     robot_mount_offset_x
     robot_mount_offset_y
+    robot_mount_offset_z
     robot_mount_offset_theta
     robot_mount_height
@@ -13,19 +12,10 @@
     robot_mount_width
     robot_base_tilt
-    pump_offset_x
-    pump_offset_y
-    pump_offset_theta
-    pump_height
-    pump_length
-    pump_width
     left_arm
     right_arm">
-  <xacro:include filename="$(find tracebot_mockup_description)/urdf/tracebot_mockup_macro.urdf.xacro"/>
   <xacro:tracebot_mockup
-    table_height="${table_height}"
-    table_length="${table_length}"
-    table_width="${table_width}"
     robot_mount_offset_x="${robot_mount_offset_x}"
     robot_mount_offset_y="${robot_mount_offset_y}"
+    robot_mount_offset_z="${robot_mount_offset_z}"
     robot_mount_offset_theta="${robot_mount_offset_theta}"
     robot_mount_height="${robot_mount_height}"
@@ -33,17 +23,8 @@
     robot_mount_width="${robot_mount_width}"
     robot_base_tilt="${robot_base_tilt}"
-    pump_offset_x="${pump_offset_x}"
-    pump_offset_y="${pump_offset_y}"
-    pump_offset_theta="${pump_offset_theta}"
-    pump_height="${pump_height}"
-    pump_length="${pump_length}"
-    pump_width="${pump_width}"
     left_arm="${left_arm}"
     right_arm="${right_arm}"
   />
-    <gazebo name="base_link">
-      <selfCollide>true</selfCollide>
-    </gazebo>
-    <gazebo name="table">
+    <gazebo name="robot_base_link">
       <selfCollide>true</selfCollide>
     </gazebo>
@@ -57,13 +38,10 @@
       <selfCollide>true</selfCollide>
     </gazebo>
-    <gazebo name="pump">
-      <selfCollide>true</selfCollide>
-    </gazebo>
-    <gazebo>
+    <!--gazebo>
       <plugin name="ros_control" filename="libgazebo_ros_control.so">
-        <!--robotNamespace>/</robotNamespace-->
-        <!--robotSimType>gazebo_ros_control/DefaultRobotHWSim</robotSimType-->
+        <!- -robotNamespace>/</robotNamespace- ->
+        <!- -robotSimType>gazebo_ros_control/DefaultRobotHWSim</robotSimType- ->
       </plugin>
-    </gazebo>
+    </gazebo-->
   </xacro:macro>
 </robot>
