Commit message: changed parameters and moved linking of arms to base from tracebot_mockup_macro to tracebot_mockup

File: tracebot_mockup_description/urdf/tracebot_mockup.urdf.xacro (robot description, xacro)
@@ -2,9 +2,9 @@
 <robot xmlns:xacro="http://wiki.ros.org/xacro" name="ur">
   <xacro:include filename="$(find tracebot_mockup_description)/urdf/tracebot_mockup_macro.urdf.xacro"/>
-  <xacro:tracebot_mockup table_length="$(arg table_length)"
-    table_width="$(arg table_width)"
-    table_height="$(arg table_height)"
+  <xacro:include filename="$(find ur_description)/urdf/ur_macro.xacro"/>
+  <xacro:tracebot_mockup
     robot_mount_offset_x="$(arg robot_mount_offset_x)"
     robot_mount_offset_y="$(arg robot_mount_offset_y)"
+    robot_mount_offset_z="$(arg robot_mount_offset_z)"
     robot_mount_offset_theta="$(arg robot_mount_offset_theta)"
     robot_mount_length="$(arg robot_mount_length)"
@@ -12,11 +12,33 @@
     robot_mount_height="$(arg robot_mount_height)"
     robot_base_tilt="$(arg robot_base_tilt)"
-    pump_offset_x="$(arg pump_offset_x)"
-    pump_offset_y="$(arg pump_offset_y)"
-    pump_offset_theta="$(arg pump_offset_theta)"
-    pump_length="$(arg pump_length)"
-    pump_width="$(arg pump_width)"
-    pump_height="$(arg pump_height)"
     left_arm="$(arg left_arm)"
     right_arm="$(arg right_arm)"/>
+  <xacro:ur_robot prefix="left_"
+    joint_limits_parameters_file="$(find ur_description)/config/$(arg left_arm)/joint_limits.yaml"
+    kinematics_parameters_file="$(find ur_description)/config/$(arg left_arm)/default_kinematics.yaml"
+    physical_parameters_file="$(find ur_description)/config/$(arg left_arm)/physical_parameters.yaml"
+    visual_parameters_file="$(find ur_description)/config/$(arg left_arm)/visual_parameters.yaml"
+    transmission_hw_interface="hardware_interface/VelocityJointInterface"
+    safety_limits="false"
+    safety_pos_margin="0.15"
+    safety_k_position="20"/>
+  <xacro:ur_robot prefix="right_"
+    joint_limits_parameters_file="$(find ur_description)/config/$(arg right_arm)/joint_limits.yaml"
+    kinematics_parameters_file="$(find ur_description)/config/$(arg right_arm)/default_kinematics.yaml"
+    physical_parameters_file="$(find ur_description)/config/$(arg right_arm)/physical_parameters.yaml"
+    visual_parameters_file="$(find ur_description)/config/$(arg right_arm)/visual_parameters.yaml"
+    transmission_hw_interface="hardware_interface/VelocityJointInterface"
+    safety_limits="false"
+    safety_pos_margin="0.15"
+    safety_k_position="20"/>
+  <joint name="left_base_link_joint" type="fixed">
+    <origin xyz="0 0 0" rpy="0 0 0"/>
+    <parent link="left_robot_mount"/>
+    <child link="left_base_link"/>
+  </joint>
+  <joint name="right_base_link_joint" type="fixed">
+    <origin xyz="0 0 0" rpy="0 0 0"/>
+    <parent link="right_robot_mount"/>
+    <child link="right_base_link"/>
+  </joint>
 </robot>

File: tracebot_mockup_description/urdf/tracebot_mockup_macro.urdf.xacro (robot description, xacro)
@@ -1,43 +1,24 @@
 <?xml version="1.0"?>
 <robot xmlns:xacro="http://wiki.ros.org/xacro">
-  <xacro:include filename="$(find ur_description)/urdf/ur_macro.xacro"/>
-  <xacro:macro name="tracebot_mockup" params="table_height
-                                              table_length
-                                              table_width
-                                              robot_mount_offset_x
-                                              robot_mount_offset_y
-                                              robot_mount_offset_theta
-                                              robot_mount_height
-                                              robot_mount_length
-                                              robot_mount_width
-                                              robot_base_tilt
-                                              pump_offset_x
-                                              pump_offset_y
-                                              pump_offset_theta
-                                              pump_height
-                                              pump_length
-                                              pump_width
-                                              left_arm
-                                              right_arm">
+  <xacro:macro name="tracebot_mockup" params="
+    robot_mount_offset_x
+    robot_mount_offset_y
+    robot_mount_offset_z
+    robot_mount_offset_theta
+    robot_mount_height
+    robot_mount_length
+    robot_mount_width
+    robot_base_tilt
+    left_arm
+    right_arm">
     <link name="base_link"/>
-    <link name="table">
-      <visual>
-        <origin xyz="0 0 0.525" rpy="0 0 0"/>
-        <geometry>
-          <mesh filename="file:///home/benrjg/astech_wss/tracebot_mockup_ws/src/tracebot_mockup/tracebot_mockup_description/meshes/table.stl" />
-        </geometry>
-        <material name="grey">
-          <color rgba="0.6 0.6 0.6 1.0"/>
-        </material>
-      </visual>
-    </link>
-    <joint name="table_joint" type="fixed">
+    <joint name="robot_mount_base_joint" type="fixed">
       <origin xyz="0 0 0" rpy="0 0 0"/>
       <parent link="base_link"/>
-      <child link="table"/>
+      <child link="robot_mount_base"/>
     </joint>
     <link name="robot_mount_base">
       <visual>
-        <origin xyz="0 0 0.6332" rpy="0 0 0"/>
+        <origin xyz="0 0 ${robot_mount_height/2}" rpy="0 0 0"/>
         <geometry>
           <mesh filename="file:///home/benrjg/astech_wss/tracebot_mockup_ws/src/tracebot_mockup/tracebot_mockup_description/meshes/stand.stl" />
@@ -48,65 +29,18 @@
       </visual>
     </link>
-    <joint name="robot_mount_base_joint" type="fixed">
-      <origin xyz="0 -0.45 0" rpy="0 0 0"/>
-      <parent link="base_link"/>
-      <child link="robot_mount_base"/>
-    </joint>
-    <link name="left_robot_mount"/>
+    <!-- Left Arm Mount -->
     <joint name="left_robot_mount_joint" type="fixed">
-      <origin xyz="-0.1293 0 1.1957" rpy="0 ${-pi/2 + robot_base_tilt} 0"/>
+      <origin xyz="${-robot_mount_offset_x} 0 ${robot_mount_height-robot_mount_offset_z}" rpy="0 ${-pi/2+robot_base_tilt} 0"/>
       <parent link="robot_mount_base"/>
       <child link="left_robot_mount"/>
     </joint>
-    <link name="right_robot_mount"/>
+    <link name="left_robot_mount"/>
+    <!-- Right Arm Mount -->
     <joint name="right_robot_mount_joint" type="fixed">
-      <origin xyz="0.1293 0 1.1957" rpy="0 ${pi/2 - robot_base_tilt} 0"/>
+      <origin xyz="${robot_mount_offset_x} 0 ${robot_mount_height-robot_mount_offset_z}" rpy="0 ${pi/2-robot_base_tilt} 0"/>
       <parent link="robot_mount_base"/>
       <child link="right_robot_mount"/>
     </joint>
-    <xacro:ur_robot prefix="left_"
-      joint_limits_parameters_file="$(find ur_description)/config/${left_arm}/joint_limits.yaml"
-                    kinematics_parameters_file="$(find ur_description)/config/${left_arm}/default_kinematics.yaml"
-                    physical_parameters_file="$(find ur_description)/config/${left_arm}/physical_parameters.yaml"
-                    visual_parameters_file="$(find ur_description)/config/${left_arm}/visual_parameters.yaml"
-                    transmission_hw_interface="hardware_interface/VelocityJointInterface"
-                    safety_limits="false"
-                    safety_pos_margin="0.15"
-                    safety_k_position="20"/>
-    <joint name="left_base_link_joint" type="fixed">
-      <origin xyz="0 0 0" rpy="0 0 0"/>
-      <parent link="left_robot_mount"/>
-      <child link="left_base_link"/>
-    </joint>
-    <xacro:ur_robot prefix="right_"
-      joint_limits_parameters_file="$(find ur_description)/config/${right_arm}/joint_limits.yaml"
-                    kinematics_parameters_file="$(find ur_description)/config/${right_arm}/default_kinematics.yaml"
-                    physical_parameters_file="$(find ur_description)/config/${right_arm}/physical_parameters.yaml"
-                    visual_parameters_file="$(find ur_description)/config/${right_arm}/visual_parameters.yaml"
-                    transmission_hw_interface="hardware_interface/VelocityJointInterface"
-                    safety_limits="false"
-                    safety_pos_margin="0.15"
-                    safety_k_position="20"/>
-    <joint name="right_base_link_joint" type="fixed">
-      <origin xyz="0 0 0" rpy="0 0 0"/>
-      <parent link="right_robot_mount"/>
-      <child link="right_base_link"/>
-    </joint>
-    <link name="pump">
-      <visual>
-        <origin xyz="0 0 0" rpy="0 0 0"/>
-        <geometry>
-          <mesh filename="file:///home/benrjg/astech_wss/tracebot_mockup_ws/src/tracebot_mockup/tracebot_mockup_description/meshes/pump.stl" />
-        </geometry>
-        <material name="pink">
-          <color rgba="1.0 0.0 1.0 1.0"/>
-        </material>
-      </visual>
-    </link>
-    <joint name="pump_joint" type="fixed">
-      <origin xyz="0 0.2 1.05" rpy="1.5708 0 0"/>
-      <parent link="table"/>
-      <child link="pump"/>
-    </joint>
+    <link name="right_robot_mount"/>
   </xacro:macro>
 </robot>

Commit message: Added updated models (and relevant parameters)

File: tracebot_mockup_description/urdf/tracebot_mockup.urdf.xacro (robot description, xacro)
@@ -2,9 +2,8 @@
 <robot xmlns:xacro="http://wiki.ros.org/xacro" name="ur">
   <xacro:include filename="$(find tracebot_mockup_description)/urdf/tracebot_mockup_macro.urdf.xacro"/>
-  <xacro:tracebot_mockup table_length="$(arg table_length)"
-    table_width="$(arg table_width)"
-    table_height="$(arg table_height)"
+  <xacro:tracebot_mockup
     robot_mount_offset_x="$(arg robot_mount_offset_x)"
     robot_mount_offset_y="$(arg robot_mount_offset_y)"
+    robot_mount_offset_z="$(arg robot_mount_offset_z)"
     robot_mount_offset_theta="$(arg robot_mount_offset_theta)"
     robot_mount_length="$(arg robot_mount_length)"
@@ -12,10 +11,4 @@
     robot_mount_height="$(arg robot_mount_height)"
     robot_base_tilt="$(arg robot_base_tilt)"
-    pump_offset_x="$(arg pump_offset_x)"
-    pump_offset_y="$(arg pump_offset_y)"
-    pump_offset_theta="$(arg pump_offset_theta)"
-    pump_length="$(arg pump_length)"
-    pump_width="$(arg pump_width)"
-    pump_height="$(arg pump_height)"
     left_arm="$(arg left_arm)"
     right_arm="$(arg right_arm)"/>

File: tracebot_mockup_description/urdf/tracebot_mockup_macro.urdf.xacro (robot description, xacro)
@@ -2,9 +2,7 @@
 <robot xmlns:xacro="http://wiki.ros.org/xacro">
   <xacro:include filename="$(find ur_description)/urdf/ur_macro.xacro"/>
-  <xacro:macro name="tracebot_mockup" params="table_height
-                                              table_length
-                                              table_width
-                                              robot_mount_offset_x
+  <xacro:macro name="tracebot_mockup" params="robot_mount_offset_x
                                               robot_mount_offset_y
+                                              robot_mount_offset_z
                                               robot_mount_offset_theta
                                               robot_mount_height
@@ -12,18 +10,13 @@
                                               robot_mount_width
                                               robot_base_tilt
-                                              pump_offset_x
-                                              pump_offset_y
-                                              pump_offset_theta
-                                              pump_height
-                                              pump_length
-                                              pump_width
                                               left_arm
                                               right_arm">
+    <!-- Base -->
     <link name="base_link"/>
-    <link name="table">
+    <link name="robot_mount_base">
       <visual>
-        <origin xyz="0 0 ${-table_height/2}" rpy="0 0 0"/>
+        <origin xyz="0 0 ${robot_mount_height/2}" rpy="0 0 0"/>
         <geometry>
-          <box size="${table_length} ${table_width} ${table_height}"/>
+          <mesh filename="file:///home/benrjg/astech_wss/tracebot_mockup_ws/src/tracebot_mockup/tracebot_mockup_description/meshes/stand.stl" />
         </geometry>
         <material name="grey">
@@ -32,46 +25,33 @@
       </visual>
     </link>
-    <joint name="table_joint" type="fixed">
-      <origin xyz="0 0 ${table_height}" rpy="0 0 0"/>
+    <joint name="robot_mount_base_joint" type="fixed">
+      <origin xyz="0 0 0" rpy="0 0 0"/>
       <parent link="base_link"/>
-      <child link="table"/>
-    </joint>
-    <link name="robot_mount_base">
-      <visual>
-        <origin xyz="0 0 ${robot_mount_height/2}" rpy="0 0 0"/>
-        <geometry>
-          <box size="${robot_mount_length} ${robot_mount_width} ${robot_mount_height}"/>
-        </geometry>
-        <material name="dark_grey">
-          <color rgba="0.4 0.4 0.4 1.0"/>
-        </material>
-      </visual>
-    </link>
-    <joint name="robot_mount_base_joint" type="fixed">
-      <origin xyz="${robot_mount_offset_x} ${robot_mount_offset_y} 0" rpy="0 0 ${robot_mount_offset_theta}"/>
-      <parent link="table"/>
       <child link="robot_mount_base"/>
     </joint>
+    <!-- Left Arm Mount -->
     <link name="left_robot_mount"/>
     <joint name="left_robot_mount_joint" type="fixed">
-      <origin xyz="${-robot_mount_length/2} 0 ${robot_mount_height/2}" rpy="0 ${-pi/2 + robot_base_tilt} 0"/>
+      <origin xyz="${-robot_mount_offset_x} 0 ${robot_mount_height-robot_mount_offset_z}" rpy="0 ${-pi/2+robot_base_tilt} 0"/>
       <parent link="robot_mount_base"/>
       <child link="left_robot_mount"/>
     </joint>
+    <!-- Right Arm Mount -->
     <link name="right_robot_mount"/>
     <joint name="right_robot_mount_joint" type="fixed">
-      <origin xyz="${robot_mount_length/2} 0 ${robot_mount_height/2}" rpy="0 ${pi/2 - robot_base_tilt} 0"/>
+      <origin xyz="${robot_mount_offset_x} 0 ${robot_mount_height-robot_mount_offset_z}" rpy="0 ${pi/2-robot_base_tilt} 0"/>
       <parent link="robot_mount_base"/>
       <child link="right_robot_mount"/>
     </joint>
+  <!--Add parameters to robot arms-->
     <xacro:ur_robot prefix="left_"
-      joint_limits_parameters_file="$(find ur_description)/config/${left_arm}/joint_limits.yaml"
-                    kinematics_parameters_file="$(find ur_description)/config/${left_arm}/default_kinematics.yaml"
-                    physical_parameters_file="$(find ur_description)/config/${left_arm}/physical_parameters.yaml"
-                    visual_parameters_file="$(find ur_description)/config/${left_arm}/visual_parameters.yaml"
-                    transmission_hw_interface="hardware_interface/VelocityJointInterface"
-                    safety_limits="false"
-                    safety_pos_margin="0.15"
-                    safety_k_position="20"/>
+      joint_limits_parameters_file="$(find ur_description)/config/$(arg left_arm)/joint_limits.yaml"
+      kinematics_parameters_file="$(find ur_description)/config/$(arg left_arm)/default_kinematics.yaml"
+      physical_parameters_file="$(find ur_description)/config/$(arg left_arm)/physical_parameters.yaml"
+      visual_parameters_file="$(find ur_description)/config/$(arg left_arm)/visual_parameters.yaml"
+      transmission_hw_interface="hardware_interface/VelocityJointInterface"
+      safety_limits="false"
+      safety_pos_margin="0.15"
+      safety_k_position="20"/>
     <joint name="left_base_link_joint" type="fixed">
       <origin xyz="0 0 0" rpy="0 0 0"/>
@@ -80,12 +60,12 @@
     </joint>
     <xacro:ur_robot prefix="right_"
-      joint_limits_parameters_file="$(find ur_description)/config/${right_arm}/joint_limits.yaml"
-                    kinematics_parameters_file="$(find ur_description)/config/${right_arm}/default_kinematics.yaml"
-                    physical_parameters_file="$(find ur_description)/config/${right_arm}/physical_parameters.yaml"
-                    visual_parameters_file="$(find ur_description)/config/${right_arm}/visual_parameters.yaml"
-                    transmission_hw_interface="hardware_interface/VelocityJointInterface"
-                    safety_limits="false"
-                    safety_pos_margin="0.15"
-                    safety_k_position="20"/>
+      joint_limits_parameters_file="$(find ur_description)/config/$(arg right_arm)/joint_limits.yaml"
+      kinematics_parameters_file="$(find ur_description)/config/$(arg right_arm)/default_kinematics.yaml"
+      physical_parameters_file="$(find ur_description)/config/$(arg right_arm)/physical_parameters.yaml"
+      visual_parameters_file="$(find ur_description)/config/$(arg right_arm)/visual_parameters.yaml"
+      transmission_hw_interface="hardware_interface/VelocityJointInterface"
+      safety_limits="false"
+      safety_pos_margin="0.15"
+      safety_k_position="20"/>
     <joint name="right_base_link_joint" type="fixed">
       <origin xyz="0 0 0" rpy="0 0 0"/>
@@ -93,20 +73,4 @@
       <child link="right_base_link"/>
     </joint>
-    <link name="pump">
-      <visual>
-        <origin xyz="0 0 ${pump_height/2}" rpy="0 0 0"/>
-        <geometry>
-          <box size="${pump_length} ${pump_width} ${pump_height}"/>
-        </geometry>
-        <material name="pink">
-          <color rgba="1.0 0.0 1.0 1.0"/>
-        </material>
-      </visual>
-    </link>
-    <joint name="pump_joint" type="fixed">
-      <origin xyz="${pump_offset_x} ${pump_offset_y} 0" rpy="0 0 ${pump_offset_theta}"/>
-      <parent link="table"/>
-      <child link="pump"/>
-    </joint>
   </xacro:macro>
 </robot>
