Commit message: Moved linking arms to base from 'macro.urdf.xacro' to standard '.urdf.xacro'

File: tracebot_mockup_description/urdf/tracebot_mockup.urdf.xacro (robot description, xacro)
@@ -1,5 +1,7 @@
 <?xml version="1.0"?>
-<robot xmlns:xacro="http://wiki.ros.org/xacro" name="ur">
+<robot xmlns:xacro="http://wiki.ros.org/xacro" name="tracebot_mockup">
   <xacro:include filename="$(find tracebot_mockup_description)/urdf/tracebot_mockup_macro.urdf.xacro"/>
+  <xacro:include filename="$(find ur_description)/urdf/ur_macro.xacro"/>
+  <!--Add parameters to robot base-->
   <xacro:tracebot_mockup
     robot_mount_offset_x="$(arg robot_mount_offset_x)"
@@ -13,3 +15,33 @@
     left_arm="$(arg left_arm)"
     right_arm="$(arg right_arm)"/>
+  <!--Add parameters to robot arms-->
+  <xacro:ur_robot prefix="left_"
+    joint_limits_parameters_file="$(find ur_description)/config/$(arg left_arm)/joint_limits.yaml"
+    kinematics_parameters_file="$(find ur_description)/config/$(arg left_arm)/default_kinematics.yaml"
+    physical_parameters_file="$(find ur_description)/config/$(arg left_arm)/physical_parameters.yaml"
+    visual_parameters_file="$(find ur_description)/config/$(arg left_arm)/visual_parameters.yaml"
+    transmission_hw_interface="hardware_interface/VelocityJointInterface"
+    safety_limits="false"
+    safety_pos_margin="0.15"
+    safety_k_position="20"/>
+  <xacro:ur_robot prefix="right_"
+    joint_limits_parameters_file="$(find ur_description)/config/$(arg right_arm)/joint_limits.yaml"
+    kinematics_parameters_file="$(find ur_description)/config/$(arg right_arm)/default_kinematics.yaml"
+    physical_parameters_file="$(find ur_description)/config/$(arg right_arm)/physical_parameters.yaml"
+    visual_parameters_file="$(find ur_description)/config/$(arg right_arm)/visual_parameters.yaml"
+    transmission_hw_interface="hardware_interface/VelocityJointInterface"
+    safety_limits="false"
+    safety_pos_margin="0.15"
+    safety_k_position="20"/>
+  <!-- Link arms to base -->
+  <joint name="left_base_link_joint" type="fixed">
+    <origin xyz="0 0 0" rpy="0 0 0"/>
+    <parent link="left_robot_mount"/>
+    <child link="left_base_link"/>
+  </joint>
+  <joint name="right_base_link_joint" type="fixed">
+    <origin xyz="0 0 0" rpy="0 0 0"/>
+    <parent link="right_robot_mount"/>
+    <child link="right_base_link"/>
+  </joint>
 </robot>

File: tracebot_mockup_description/urdf/tracebot_mockup_macro.urdf.xacro (robot description, xacro)
@@ -1,5 +1,4 @@
 <?xml version="1.0"?>
 <robot xmlns:xacro="http://wiki.ros.org/xacro">
-  <xacro:include filename="$(find ur_description)/urdf/ur_macro.xacro"/>
   <xacro:macro name="tracebot_mockup" params="robot_mount_offset_x
                                               robot_mount_offset_y
@@ -14,4 +13,9 @@
     <!-- Base -->
     <link name="base_link"/>
+    <joint name="robot_mount_base_joint" type="fixed">
+      <origin xyz="0 0 0" rpy="0 0 0"/>
+      <parent link="base_link"/>
+      <child link="robot_mount_base"/>
+    </joint>
     <link name="robot_mount_base">
       <visual>
@@ -25,11 +29,5 @@
       </visual>
     </link>
-    <joint name="robot_mount_base_joint" type="fixed">
-      <origin xyz="0 0 0" rpy="0 0 0"/>
-      <parent link="base_link"/>
-      <child link="robot_mount_base"/>
-    </joint>
     <!-- Left Arm Mount -->
-    <link name="left_robot_mount"/>
     <joint name="left_robot_mount_joint" type="fixed">
       <origin xyz="${-robot_mount_offset_x} 0 ${robot_mount_height-robot_mount_offset_z}" rpy="0 ${-pi/2+robot_base_tilt} 0"/>
@@ -37,6 +35,6 @@
       <child link="left_robot_mount"/>
     </joint>
+    <link name="left_robot_mount"/>
     <!-- Right Arm Mount -->
-    <link name="right_robot_mount"/>
     <joint name="right_robot_mount_joint" type="fixed">
       <origin xyz="${robot_mount_offset_x} 0 ${robot_mount_height-robot_mount_offset_z}" rpy="0 ${pi/2-robot_base_tilt} 0"/>
@@ -44,33 +42,5 @@
       <child link="right_robot_mount"/>
     </joint>
-  <!--Add parameters to robot arms-->
-    <xacro:ur_robot prefix="left_"
-      joint_limits_parameters_file="$(find ur_description)/config/$(arg left_arm)/joint_limits.yaml"
-      kinematics_parameters_file="$(find ur_description)/config/$(arg left_arm)/default_kinematics.yaml"
-      physical_parameters_file="$(find ur_description)/config/$(arg left_arm)/physical_parameters.yaml"
-      visual_parameters_file="$(find ur_description)/config/$(arg left_arm)/visual_parameters.yaml"
-      transmission_hw_interface="hardware_interface/VelocityJointInterface"
-      safety_limits="false"
-      safety_pos_margin="0.15"
-      safety_k_position="20"/>
-    <joint name="left_base_link_joint" type="fixed">
-      <origin xyz="0 0 0" rpy="0 0 0"/>
-      <parent link="left_robot_mount"/>
-      <child link="left_base_link"/>
-    </joint>
-    <xacro:ur_robot prefix="right_"
-      joint_limits_parameters_file="$(find ur_description)/config/$(arg right_arm)/joint_limits.yaml"
-      kinematics_parameters_file="$(find ur_description)/config/$(arg right_arm)/default_kinematics.yaml"
-      physical_parameters_file="$(find ur_description)/config/$(arg right_arm)/physical_parameters.yaml"
-      visual_parameters_file="$(find ur_description)/config/$(arg right_arm)/visual_parameters.yaml"
-      transmission_hw_interface="hardware_interface/VelocityJointInterface"
-      safety_limits="false"
-      safety_pos_margin="0.15"
-      safety_k_position="20"/>
-    <joint name="right_base_link_joint" type="fixed">
-      <origin xyz="0 0 0" rpy="0 0 0"/>
-      <parent link="right_robot_mount"/>
-      <child link="right_base_link"/>
-    </joint>
+    <link name="right_robot_mount"/>
   </xacro:macro>
 </robot>

Commit message: updated README with changed parameters and image

File: tracebot_mockup_description/urdf/tracebot_mockup.urdf.xacro (robot description, xacro)
@@ -36,10 +36,10 @@
   <!-- Link arms to base -->
   <joint name="left_base_link_joint" type="fixed">
-    <origin xyz="0 0 0" rpy="0 0 0"/>
+    <origin xyz="0 0 0" rpy="0 0 1.5708"/>
     <parent link="left_robot_mount"/>
     <child link="left_base_link"/>
   </joint>
   <joint name="right_base_link_joint" type="fixed">
-    <origin xyz="0 0 0" rpy="0 0 0"/>
+    <origin xyz="0 0 0" rpy="0 0 -1.5708"/>
     <parent link="right_robot_mount"/>
     <child link="right_base_link"/>

Commit message: Added camera mount to robot base

File: tracebot_mockup_description/urdf/tracebot_mockup.urdf.xacro (robot description, xacro)
@@ -14,5 +14,6 @@
     robot_base_tilt="$(arg robot_base_tilt)"
     left_arm="$(arg left_arm)"
-    right_arm="$(arg right_arm)"/>
+    right_arm="$(arg right_arm)"
+    camera_mount_offset_z="$(arg camera_mount_offset_z)"/>
   <!--Add parameters to robot arms-->
   <xacro:ur_robot prefix="left_"
@@ -45,3 +46,9 @@
     <child link="right_base_link"/>
   </joint>
+  <!-- Link camera to base -->
+  <!--joint name="camera_base_link_joint" type="fixed">
+    <origin xyz="0 0 0" rpy="0 0 0"/>
+    <parent link="camera_mount"/>
+    <child link="camera_base_link"/>
+  </joint-->
 </robot>

File: tracebot_mockup_description/urdf/tracebot_mockup_macro.urdf.xacro (robot description, xacro)
@@ -10,5 +10,6 @@
                                               robot_base_tilt
                                               left_arm
-                                              right_arm">
+                                              right_arm
+                                              camera_mount_offset_z">
     <!-- Base -->
     <link name="base_link"/>
@@ -43,4 +44,11 @@
     </joint>
     <link name="right_robot_mount"/>
+    <!-- Camera Mount -->
+    <joint name="camera_mount_joint" type="fixed">
+      <origin xyz="0 0 ${robot_mount_height+camera_mount_offset_z}" rpy="0 0 0"/>
+      <parent link="robot_mount_base"/>
+      <child link="camera_mount"/>
+    </joint>
+    <link name="camera_mount"/>
   </xacro:macro>
 </robot>

Commit message: Added realsense camera to Rviz model

File: tracebot_mockup_description/urdf/tracebot_mockup.urdf.xacro (robot description, xacro)
@@ -46,9 +46,3 @@
     <child link="right_base_link"/>
   </joint>
-  <!-- Link camera to base -->
-  <!--joint name="camera_base_link_joint" type="fixed">
-    <origin xyz="0 0 0" rpy="0 0 0"/>
-    <parent link="camera_mount"/>
-    <child link="camera_base_link"/>
-  </joint-->
 </robot>

File: tracebot_mockup_description/urdf/tracebot_mockup_macro.urdf.xacro (robot description, xacro)
@@ -45,4 +45,5 @@
     <link name="right_robot_mount"/>
     <!-- Camera Mount -->
+    <xacro:include filename="$(find realsense2_description)/urdf/_d435.urdf.xacro" />
     <joint name="camera_mount_joint" type="fixed">
       <origin xyz="0 0 ${robot_mount_height+camera_mount_offset_z}" rpy="0 0 0"/>
@@ -51,4 +52,9 @@
     </joint>
     <link name="camera_mount"/>
+    <xacro:sensor_d435 parent="camera_mount"
+      use_nominal_extrinsics="false"
+      add_plug="false" use_mesh="true">
+      <origin xyz="0 0 0" rpy="0 0.785398 1.5708"/>
+    </xacro:sensor_d435>
   </xacro:macro>
 </robot>

Commit message: added 'tilt' parameter for camera

File: tracebot_mockup_description/urdf/tracebot_mockup.urdf.xacro (robot description, xacro)
@@ -15,4 +15,5 @@
     left_arm_model="$(arg left_arm_model)"
     right_arm_model="$(arg right_arm_model)"
-    camera_mount_offset_z="$(arg camera_mount_offset_z)"/>
+    camera_mount_offset_z="$(arg camera_mount_offset_z)"
+    camera_tilt="$(arg camera_tilt)"/>
 </robot>

File: tracebot_mockup_description/urdf/tracebot_mockup_macro.urdf.xacro (robot description, xacro)
@@ -12,5 +12,6 @@
                                               left_arm_model
                                               right_arm_model
-                                              camera_mount_offset_z">
+                                              camera_mount_offset_z
+                                              camera_tilt">
     <!-- Base -->
     <link name="${robot_name}_base_link"/>
@@ -87,6 +88,6 @@
       add_plug="false"
       use_mesh="true"
-      name="camera">
-      <origin xyz="0 0 0" rpy="0 0.785398 1.5708"/>
+      name="${robot_name}_camera">
+      <origin xyz="0 0 0" rpy="0 ${camera_tilt} 1.5708"/>
     </xacro:sensor_d435>
   </xacro:macro>

File: tracebot_mockup_gazebo/urdf/tracebot_mockup.urdf.xacro (robot description, xacro)
@@ -15,4 +15,5 @@
   <xacro:arg name="right_arm_model" default="ur5e"/>
   <xacro:arg name="camera_mount_offset_z" default="0.65169"/>
+  <xacro:arg name="camera_tilt" default="0.785398"/>
   <!--Robot arm parameters-->
   <xacro:arg name="transmission_hw_interface" default="hardware_interface/PositionJointInterface"/>
@@ -30,5 +31,6 @@
     left_arm_model="$(arg left_arm_model)"
     right_arm_model="$(arg right_arm_model)"
-    camera_mount_offset_z="$(arg camera_mount_offset_z)"/>
+    camera_mount_offset_z="$(arg camera_mount_offset_z)"
+    camera_tilt="$(arg camera_tilt)"/>
   <!--Link base to world-->
   <link name="world"/>
@@ -47,10 +49,10 @@
   <xacro:include filename="$(find tracebot_mockup_gazebo)/urdf/_d435.gazebo.xacro"/>
   <xacro:gazebo_d435
-    camera_name="camera"
-    reference_link="camera_link"
-    topics_ns="camera"
-    depth_optical_frame="camera_depth_optical_frame"
-    color_optical_frame="camera_color_optical_frame"
-    infrared1_optical_frame="camera_left_ir_optical_frame"
-    infrared2_optical_frame="camera_right_ir_optical_frame"/>
+    camera_name="$(arg robot_name)_camera"
+    reference_link="$(arg robot_name)_camera_link"
+    topics_ns="$(arg robot_name)_camera"
+    depth_optical_frame="$(arg robot_name)_camera_depth_optical_frame"
+    color_optical_frame="$(arg robot_name)_camera_color_optical_frame"
+    infrared1_optical_frame="$(arg robot_name)_camera_left_ir_optical_frame"
+    infrared2_optical_frame="$(arg robot_name)_camera_right_ir_optical_frame"/>
 </robot>

File: tracebot_mockup_gazebo/urdf/tracebot_mockup_macro.urdf.xacro (robot description, xacro)
@@ -12,5 +12,6 @@
                                                      left_arm_model
                                                      right_arm_model
-                                                     camera_mount_offset_z">
+                                                     camera_mount_offset_z
+                                                     camera_tilt">
     <xacro:include filename="$(find tracebot_mockup_description)/urdf/tracebot_mockup_macro.urdf.xacro"/>
     <!--Pass arguments to tracebot_mockup-->
@@ -28,4 +29,5 @@
       right_arm_model="$(arg right_arm_model)"
       camera_mount_offset_z="${camera_mount_offset_z}"
+      camera_tilt="${camera_tilt}"
     />
     <!-- Configure self collision properties per link -->
