Commit message: Swap left<->right prefixes

File: tracebot_mockup_description/urdf/tracebot_mockup_macro.urdf.xacro (robot description, xacro)
@@ -53,5 +53,5 @@
     <link name="left_robot_mount"/>
     <joint name="left_robot_mount_joint" type="fixed">
-      <origin xyz="${robot_mount_length/2} 0 ${robot_mount_height/2}" rpy="0 ${pi/2 - robot_base_tilt} 0"/>
+      <origin xyz="${-robot_mount_length/2} 0 ${robot_mount_height/2}" rpy="0 ${-pi/2 + robot_base_tilt} 0"/>
       <parent link="robot_mount_base"/>
       <child link="left_robot_mount"/>
@@ -59,5 +59,5 @@
     <link name="right_robot_mount"/>
     <joint name="right_robot_mount_joint" type="fixed">
-      <origin xyz="${-robot_mount_length/2} 0 ${robot_mount_height/2}" rpy="0 ${-pi/2 + robot_base_tilt} 0"/>
+      <origin xyz="${robot_mount_length/2} 0 ${robot_mount_height/2}" rpy="0 ${pi/2 - robot_base_tilt} 0"/>
       <parent link="robot_mount_base"/>
       <child link="right_robot_mount"/>

Commit message: Added table, stand and pump models to RViz

File: tracebot_mockup_description/urdf/tracebot_mockup_macro.urdf.xacro (robot description, xacro)
@@ -23,7 +23,7 @@
     <link name="table">
       <visual>
-        <origin xyz="0 0 ${-table_height/2}" rpy="0 0 0"/>
+        <origin xyz="0 0 0.525" rpy="0 0 0"/>
         <geometry>
-          <box size="${table_length} ${table_width} ${table_height}"/>
+          <mesh filename="file:///home/benrjg/astech_wss/tracebot_mockup_ws/src/tracebot_mockup/tracebot_mockup_description/meshes/table.stl" />
         </geometry>
         <material name="grey">
@@ -33,5 +33,5 @@
     </link>
     <joint name="table_joint" type="fixed">
-      <origin xyz="0 0 ${table_height}" rpy="0 0 0"/>
+      <origin xyz="0 0 0" rpy="0 0 0"/>
       <parent link="base_link"/>
       <child link="table"/>
@@ -39,21 +39,21 @@
     <link name="robot_mount_base">
       <visual>
-        <origin xyz="0 0 ${robot_mount_height/2}" rpy="0 0 0"/>
+        <origin xyz="0 0 0.6332" rpy="0 0 0"/>
         <geometry>
-          <box size="${robot_mount_length} ${robot_mount_width} ${robot_mount_height}"/>
+          <mesh filename="file:///home/benrjg/astech_wss/tracebot_mockup_ws/src/tracebot_mockup/tracebot_mockup_description/meshes/stand.stl" />
         </geometry>
-        <material name="dark_grey">
-          <color rgba="0.4 0.4 0.4 1.0"/>
+        <material name="grey">
+          <color rgba="0.6 0.6 0.6 1.0"/>
         </material>
       </visual>
     </link>
     <joint name="robot_mount_base_joint" type="fixed">
-      <origin xyz="${robot_mount_offset_x} ${robot_mount_offset_y} 0" rpy="0 0 ${robot_mount_offset_theta}"/>
-      <parent link="table"/>
+      <origin xyz="0 -0.45 0" rpy="0 0 0"/>
+      <parent link="base_link"/>
       <child link="robot_mount_base"/>
     </joint>
     <link name="left_robot_mount"/>
     <joint name="left_robot_mount_joint" type="fixed">
-      <origin xyz="${-robot_mount_length/2} 0 ${robot_mount_height/2}" rpy="0 ${-pi/2 + robot_base_tilt} 0"/>
+      <origin xyz="-0.1293 0 1.1957" rpy="0 ${-pi/2 + robot_base_tilt} 0"/>
       <parent link="robot_mount_base"/>
       <child link="left_robot_mount"/>
@@ -61,5 +61,5 @@
     <link name="right_robot_mount"/>
     <joint name="right_robot_mount_joint" type="fixed">
-      <origin xyz="${robot_mount_length/2} 0 ${robot_mount_height/2}" rpy="0 ${pi/2 - robot_base_tilt} 0"/>
+      <origin xyz="0.1293 0 1.1957" rpy="0 ${pi/2 - robot_base_tilt} 0"/>
       <parent link="robot_mount_base"/>
       <child link="right_robot_mount"/>
@@ -95,7 +95,7 @@
     <link name="pump">
       <visual>
-        <origin xyz="0 0 ${pump_height/2}" rpy="0 0 0"/>
+        <origin xyz="0 0 0" rpy="0 0 0"/>
         <geometry>
-          <box size="${pump_length} ${pump_width} ${pump_height}"/>
+          <mesh filename="file:///home/benrjg/astech_wss/tracebot_mockup_ws/src/tracebot_mockup/tracebot_mockup_description/meshes/pump.stl" />
         </geometry>
         <material name="pink">
@@ -105,5 +105,5 @@
     </link>
     <joint name="pump_joint" type="fixed">
-      <origin xyz="${pump_offset_x} ${pump_offset_y} 0" rpy="0 0 ${pump_offset_theta}"/>
+      <origin xyz="0 0.2 1.05" rpy="1.5708 0 0"/>
       <parent link="table"/>
       <child link="pump"/>

Commit message: Added gazebo model for tracebot

File: tracebot_mockup_description/urdf/tracebot_mockup_macro.urdf.xacro (robot description, xacro)
@@ -2,22 +2,23 @@
 <robot xmlns:xacro="http://wiki.ros.org/xacro">
   <xacro:include filename="$(find ur_description)/urdf/ur_macro.xacro"/>
-  <xacro:macro name="tracebot_mockup" params="table_height
-                                              table_length
-                                              table_width
-                                              robot_mount_offset_x
-                                              robot_mount_offset_y
-                                              robot_mount_offset_theta
-                                              robot_mount_height
-                                              robot_mount_length
-                                              robot_mount_width
-                                              robot_base_tilt
-                                              pump_offset_x
-                                              pump_offset_y
-                                              pump_offset_theta
-                                              pump_height
-                                              pump_length
-                                              pump_width
-                                              left_arm
-                                              right_arm">
+  <xacro:macro name="tracebot_mockup"
+    params="table_height
+    table_length
+    table_width
+    robot_mount_offset_x
+    robot_mount_offset_y
+    robot_mount_offset_theta
+    robot_mount_height
+    robot_mount_length
+    robot_mount_width
+    robot_base_tilt
+    pump_offset_x
+    pump_offset_y
+    pump_offset_theta
+    pump_height
+    pump_length
+    pump_width
+    left_arm
+    right_arm">
     <link name="base_link"/>
     <link name="table">
@@ -55,5 +56,5 @@
     <link name="left_robot_mount"/>
     <joint name="left_robot_mount_joint" type="fixed">
-      <origin xyz="-0.1293 0 1.1957" rpy="0 ${-pi/2 + robot_base_tilt} 0"/>
+      <origin xyz="-0.1293 0 1.1957" rpy="0 ${-1.57079632679+robot_base_tilt} 0"/>
       <parent link="robot_mount_base"/>
       <child link="left_robot_mount"/>
@@ -61,5 +62,5 @@
     <link name="right_robot_mount"/>
     <joint name="right_robot_mount_joint" type="fixed">
-      <origin xyz="0.1293 0 1.1957" rpy="0 ${pi/2 - robot_base_tilt} 0"/>
+      <origin xyz="0.1293 0 1.1957" rpy="0 ${1.57079632679-robot_base_tilt} 0"/>
       <parent link="robot_mount_base"/>
       <child link="right_robot_mount"/>

Commit message: Added functionality to arms in gazebo

File: tracebot_mockup_description/urdf/tracebot_mockup_macro.urdf.xacro (robot description, xacro)
@@ -1,15 +1,14 @@
 <?xml version="1.0"?>
 <robot xmlns:xacro="http://wiki.ros.org/xacro">
-  <xacro:macro name="tracebot_mockup" params="
-    robot_mount_offset_x
-    robot_mount_offset_y
-    robot_mount_offset_z
-    robot_mount_offset_theta
-    robot_mount_height
-    robot_mount_length
-    robot_mount_width
-    robot_base_tilt
-    left_arm
-    right_arm">
+  <xacro:macro name="tracebot_mockup" params="robot_mount_offset_x
+                                              robot_mount_offset_y
+                                              robot_mount_offset_z
+                                              robot_mount_offset_theta
+                                              robot_mount_height
+                                              robot_mount_length
+                                              robot_mount_width
+                                              robot_base_tilt
+                                              left_arm
+                                              right_arm">
     <link name="base_link"/>
     <joint name="robot_mount_base_joint" type="fixed">

Commit message: Updated mesh file location

File: tracebot_mockup_description/urdf/tracebot_mockup_macro.urdf.xacro (robot description, xacro)
@@ -22,5 +22,5 @@
         <origin xyz="0 0 ${robot_mount_height/2}" rpy="0 0 0"/>
         <geometry>
-          <mesh filename="file:///home/benrjg/astech_wss/tracebot_mockup_ws/src/tracebot_mockup/tracebot_mockup_description/meshes/stand.stl" />
+          <mesh filename="package://tracebot_mockup_description/meshes/stand.stl" />
         </geometry>
         <material name="grey">

Commit message: (Non Functional) started work on realsense ros/gazebo plugin

File: tracebot_mockup_description/urdf/tracebot_mockup_macro.urdf.xacro (robot description, xacro)
@@ -54,5 +54,7 @@
     <xacro:sensor_d435 parent="camera_mount"
       use_nominal_extrinsics="false"
-      add_plug="false" use_mesh="true">
+      add_plug="false"
+      use_mesh="true"
+      name="tracebot_camera">
       <origin xyz="0 0 0" rpy="0 0.785398 1.5708"/>
     </xacro:sensor_d435>

File: tracebot_mockup_gazebo/urdf/tracebot_mockup_macro.urdf.xacro (robot description, xacro)
@@ -14,4 +14,5 @@
     camera_mount_offset_z">
     <xacro:include filename="$(find tracebot_mockup_description)/urdf/tracebot_mockup_macro.urdf.xacro"/>
+    <!--xacro:include filename="$(find tracebot_macro_gazebo)/urdf/_d435.gazebo.xacro"/-->
     <!--Pass arguments to tracebot_mockup-->
     <xacro:tracebot_mockup
@@ -32,4 +33,13 @@
       <selfCollide>true</selfCollide>
     </gazebo>
-  </xacro:macro>
+    <!-- Gazebo Plugins -->
+    <!--xacro:gazebo_d435
+      camera_name="${camera_name}"
+      reference_link="${camera_name}_link"
+      topics_ns="${topics_ns}"
+      depth_optical_frame="${camera_name}_depth_optical_frame"
+      color_optical_frame="${camera_name}_color_optical_frame"
+      infrared1_optical_frame="${camera_name}_left_ir_optical_frame"
+      infrared2_optical_frame="${camera_name}_right_ir_optical_frame"/>
+  </xacro:macro-->
 </robot>

Commit message: Updated camera links/joints to include robot_name

File: tracebot_mockup_description/urdf/tracebot_mockup_macro.urdf.xacro (robot description, xacro)
@@ -77,15 +77,15 @@
     <!-- Camera Mount -->
     <xacro:include filename="$(find realsense2_description)/urdf/_d435.urdf.xacro" />
-    <joint name="camera_mount_joint" type="fixed">
+    <joint name="${robot_name}_camera_mount_joint" type="fixed">
       <origin xyz="0 0 ${mount_base_height+camera_mount_offset_z}" rpy="0 0 0"/>
       <parent link="${robot_name}_arm_mount_base"/>
-      <child link="camera_mount"/>
+      <child link="${robot_name}_camera_mount"/>
     </joint>
-    <link name="camera_mount"/>
-    <xacro:sensor_d435 parent="camera_mount"
+    <link name="${robot_name}_camera_mount"/>
+    <xacro:sensor_d435 parent="${robot_name}_camera_mount"
       use_nominal_extrinsics="false"
       add_plug="false"
       use_mesh="true"
-      name="tracebot_camera">
+      name="${robot_name}_camera">
       <origin xyz="0 0 0" rpy="0 0.785398 1.5708"/>
     </xacro:sensor_d435>

File: tracebot_mockup_gazebo/urdf/tracebot_mockup.urdf.xacro (robot description, xacro)
@@ -45,3 +45,11 @@
     </plugin>
   </gazebo>
+  <!--xacro:gazebo_d435
+    camera_name="${robot_name}_camera"
+    reference_link="${robot_name}_camera_link"
+    topics_ns="${topics_ns}"
+    depth_optical_frame="${robot_name}_camera_depth_optical_frame"
+    color_optical_frame="${robot_name}_camera_color_optical_frame"
+    infrared1_optical_frame="${robot_name}_camera_left_ir_optical_frame"
+    infrared2_optical_frame="${robot_name}_camera_right_ir_optical_frame"/-->
 </robot>

File: tracebot_mockup_gazebo/urdf/tracebot_mockup_macro.urdf.xacro (robot description, xacro)
@@ -79,13 +79,4 @@
       <selfCollide>true</selfCollide>
     </gazebo>
-    <!-- Gazebo Plugins -->
-    <!--xacro:gazebo_d435
-      camera_name="${camera_name}"
-      reference_link="${camera_name}_link"
-      topics_ns="${topics_ns}"
-      depth_optical_frame="${camera_name}_depth_optical_frame"
-      color_optical_frame="${camera_name}_color_optical_frame"
-      infrared1_optical_frame="${camera_name}_left_ir_optical_frame"
-      infrared2_optical_frame="${camera_name}_right_ir_optical_frame"/-->
   </xacro:macro>
 </robot>

Commit message: Fixed incorrect filepath

File: tracebot_mockup_description/urdf/tracebot_mockup_macro.urdf.xacro (robot description, xacro)
@@ -23,5 +23,5 @@
         <origin xyz="0 0 ${robot_mount_height/2}" rpy="0 0 0"/>
         <geometry>
-          <mesh filename="file:///home/benrjg/astech_wss/tracebot_mockup_ws/src/tracebot_mockup/tracebot_mockup_description/meshes/stand.stl" />
+          <mesh filename="package://tracebot_mockup_description/meshes/stand.stl" />
         </geometry>
         <material name="grey">
